Commit message: More work on Hw0

File: src/hw0/RRPbot.urdf (robot description, URDF)
Before this commit: robot RRPbot, 2 links, 1 joints
Links:
- added link link1, mass 0.01; visual sphere radius=0.2
- added link link2, mass 0.01; visual sphere radius=0.2
- link base_link: mass 0 -> 0.01; geometry 
- link link0: mass 0 -> 0.01
Joints:
- added joint j1: type revolute, parent link0, child link1, origin xyz=0.000000 0.000000 0.500000 rpy=1.5708 0.000000 -0.000000, axis 0 0 1, limit lower=-2.967 upper=2.967 effort=176 velocity=1.7104
- added joint j2: type prismatic, parent link1, child link2, origin xyz=0.000000 0.000000 0.000000 rpy=-1.5708 0.000000 -0.000000, axis 0 0 1, limit lower=-2.967 upper=2.967 effort=176 velocity=1.7104
- joint j0: origin xyz=0.000000 0.000000 2.000000 rpy=-0.000000 0.000000 -0.000000 -> xyz=0.000000 0.000000 0.000000 rpy=-0.000000 0.000000 -0.000000; type prismatic -> revolute

Commit message: updating urdf filepaths temporarily

File: src/hw0/RRPbot.urdf (robot description, URDF)
Before this commit: robot RRPbot, 4 links, 3 joints
Links:
- link base_link: geometry visual box size=0.2 0.2 0.2

Commit message: changed robot graphics

File: src/hw0/RRPbot.urdf (robot description, URDF)
Before this commit: robot RRPbot, 4 links, 3 joints
Links:
- link link0: geometry visual box size=0.1 0.1 0.15; visual cylinder length=0.05 radius=0.1
- link link2: mass 0.01 -> 1
Joints:
- joint j1: origin xyz=0.000000 0.000000 0.4250000 rpy=1.5708 0.000000 -0.000000 -> xyz=0.000000 0.000000 0.20000 rpy=1.5708 0.000000 -0.000000
