Commit message: Updated kuka urdf

File: src/demo_project/kuka_iiwa.urdf (robot description, URDF)
Before this commit: robot kuka_iiwa, 8 links, 7 joints
Joints:
- joint j0: origin xyz=0.000000 0.000000 0.155767 rpy=-0.000000 0.000000 -0.000000 -> xyz=0.000000 0.000000 0.155767 rpy=0.000000 0.000000 0.000000
- joint j1: origin xyz=0.000000 0.000000 0.182500 rpy=-0.000000 0.000000 -0.000000 -> xyz=0.000000 0.000000 0.182500 rpy=0.000000 0.000000 0.000000
- joint j2: origin xyz=0.000000 0.000000 0.185000 rpy=-0.000000 0.000000 -0.000000 -> xyz=0.000000 0.000000 0.185000 rpy=0.000000 0.000000 0.000000
- joint j3: origin xyz=0.000000 0.000000 0.217000 rpy=-0.000000 0.000000 -0.000000 -> xyz=0.000000 0.000000 0.217000 rpy=0.000000 0.000000 3.1415926535897
- joint j4: origin xyz=0.000000 0.000000 0.186000 rpy=-0.000000 0.000000 -0.000000 -> xyz=0.000000 0.000000 0.186000 rpy=0.000000 0.000000 -3.1415926535897
- joint j5: origin xyz=0.000000 0.000000 0.217003 rpy=-0.000000 0.000000 -0.000000 -> xyz=0.000000 0.000000 0.217003 rpy=0.000000 0.000000 0.000000
- joint j6: origin xyz=0.000000 0.000000 0.081000 rpy=-0.000000 0.000000 -0.000000 -> xyz=0.000000 0.000000 0.081000 rpy=0.000000 0.000000 0.000000
