Commit message: Sawyer update!

File: src/sawyer/sawyer.urdf (robot description, URDF)
Before this commit: robot sawyer, 24 links, 23 joints
Links:
- removed link controller_box
- removed link head_camera
- removed link pedestal
- removed link pedestal_feet
- removed link right_arm_itb
- removed link right_hand
- removed link right_hand_camera
- removed link right_l1_2
- removed link right_l2_2
- removed link right_l4_2
- removed link right_torso_itb
- removed link right_wrist
- removed link screen
- removed link torso
- link base: mass 34.4 -> 60.86397744; geometry visual mesh filename=meshes/pedestal.obj
Joints:
- removed joint controller_box_fixed
- removed joint display_joint
- removed joint head_camera
- removed joint pedestal_feet_fixed
- removed joint pedestal_fixed
- removed joint right_arm_itb
- removed joint right_hand
- removed joint right_hand_camera
- removed joint right_j1_2
- removed joint right_j2_2
- removed joint right_j4_2
- removed joint right_torso_itb
- removed joint right_wrist
- removed joint torso_t0
- joint head_pan: type revolute -> fixed
- joint right_j2: origin xyz=0 -0.14 0.1425 rpy=1.57079632679 0 0 -> xyz=0 -0.14 0.1325 rpy=1.57079632679 0 0

Commit message: Linking graphics

File: src/sawyer/sawyer.urdf (robot description, URDF)
Before this commit: robot sawyer, 10 links, 9 joints
Links:
- link base: geometry visual mesh filename=sawyer_graphics/pedestal.obj
- link head: geometry visual mesh filename=sawyer_graphics/head.obj
- link right_arm_base_link: geometry visual mesh filename=sawyer_graphics/base.obj
- link right_l0: geometry visual mesh filename=sawyer_graphics/l0.obj
- link right_l1: geometry visual mesh filename=sawyer_graphics/l1.obj
- link right_l2: geometry visual mesh filename=sawyer_graphics/l2.obj
- link right_l3: geometry visual mesh filename=sawyer_graphics/l3.obj
- link right_l4: geometry visual mesh filename=sawyer_graphics/l4.obj
- link right_l5: geometry visual mesh filename=sawyer_graphics/l5.obj
- link right_l6: geometry visual mesh filename=sawyer_graphics/l6.obj
