Commit message: Updating with newer puma branch

File: src/puma/puma.urdf (robot description, URDF)
Before this commit: robot puma, 7 links, 6 joints
Links:
- link end-effector: mass 1.0 -> 0.09
Joints:
- joint elbow: limit lower=-3.14159 upper=3.14159 effort=89.4 velocity=1.0 -> lower=-0.69813 upper=4.18879 effort=89.4 velocity=1.0
- joint shoulder-pitch: limit lower=-3.14159 upper=3.14159 effort=186.4 velocity=1.0 -> lower=-3.89208 upper=0.75049 effort=186.4 velocity=1.0; origin xyz=0.0 0.2435 0.0 rpy=-1.5707963268 0.0 0.0 -> xyz=0.0 0.2435 0.0 rpy=-1.57079632679489661923 0.0 0.0
- joint shoulder-yaw: origin xyz=0.0 0.0 0.66 rpy=0.0 0.0 0.0 -> xyz=0.0 0.0 0.0 rpy=0.0 0.0 0.0
- joint wrist-pitch: limit lower=-3.14159 upper=3.14159 effort=20.1 velocity=1.0 -> lower=-1.74532 upper=1.74532 effort=20.1 velocity=1.0; origin xyz=0.0 0.0 0.0 rpy=0.0 1.5707963268 -3.1415926536 -> xyz=0.0 0.0 0.0 rpy=-1.57079632679489661923 0.0 0.0
- joint wrist-roll1: origin xyz=-0.0203 -0.4331 0.0 rpy=1.5707963268 0.0 0.0 -> xyz=-0.0203 -0.4331 0.0 rpy=1.57079632679489661923 0.0 0.0
- joint wrist-roll2: limit lower=-3.14159 upper=3.14159 effort=21.3 velocity=1.0 -> lower=-4.64257 upper=4.64257 effort=21.3 velocity=1.0; origin xyz=-0.07 0.0 0.0 rpy=1.5707963268 0.0 0.0 -> xyz=0.0 -0.16 0.0 rpy=1.57079632679489661923 0.0 0.0
